Commit message: cup manipulator working

File: model_using_onshape_to_robot/cup_manipulator/cup_manipulator_obj.urdf (robot description, URDF)
Before this commit: robot cup_manipulator, 4 links, 3 joints
Links:
- removed link part_1
- link link2: geometry collision mesh filename=package://assets/link2.obj; collision mesh filename=package://assets/simple_ball.obj
Joints:
- removed joint cup_ee
- removed joint link1_mount
- added joint link1_base: type revolute, parent base_mount_manipulator, child link1, origin xyz=0 -2.53063e-17 1.17625 rpy=3.14159 -0 0, axis 0 0 1, limit lower=-3.141592653589793 upper=3.141592653589793 effort=10 velocity=10
- joint link2_link1: origin xyz=-0.953 -5.07838e-17 -0.118125 rpy=3.14159 -0 0.526654 -> xyz=-0.953 4.89859e-18 0.118125 rpy=0 -0 0

File: model_using_onshape_to_robot/cup_manipulator/cup_manipulator_obj_v2.urdf (robot description, URDF)
Before this commit: robot cup_manipulator, 3 links, 2 joints
Links:
- link base_mount_manipulator: geometry collision mesh filename=package://cup_assets/base_mount_manipulator.obj; visual mesh filename=package://cup_assets/base_mount_manipulator.obj
- link link1: geometry collision mesh filename=package://cup_assets/link1.obj; visual mesh filename=package://cup_assets/link1.obj
- link link2: geometry collision mesh filename=package://cup_assets/link2.obj; collision mesh filename=package://cup_assets/part_1.obj
Joints:
- joint link1_base: origin xyz=0 -2.53063e-17 1.17625 rpy=3.14159 -0 0 -> xyz=0 -3.91841e-17 1.17625 rpy=3.14159 -0 0
- joint link2_link1: origin xyz=-0.953 4.89859e-18 0.118125 rpy=0 -0 0 -> xyz=0.953 1.87764e-17 -0.08 rpy=0 -0 3.14159

File: model_using_onshape_to_robot/cup_manipulator/cup_manipulator_v1.urdf (robot description, URDF)
Before this commit: robot cup_manipulator, 3 links, 2 joints
Links:
- added link part_1, mass 1e-09; collision mesh filename=package://assets/part_1.stl; visual mesh filename=package://assets/part_1.stl
- link link2: geometry collision mesh filename=package://assets/link2.stl; visual mesh filename=package://assets/link2.stl
Joints:
- removed joint link1_base
- added joint cup_ee: type revolute, parent link2, child part_1, origin xyz=-0.953 -2.22045e-16 0 rpy=0 -0 -2.98756, axis 0 0 1, limit lower=-3.141592653589793 upper=3.141592653589793 effort=10 velocity=10
- added joint link1_mount: type revolute, parent base_mount_manipulator, child link1, origin xyz=-6.45044e-17 1.47663e-17 1.17625 rpy=0 -0 2.04171, axis 0 0 1, limit lower=-3.141592653589793 upper=3.141592653589793 effort=10 velocity=10
- joint link2_link1: origin xyz=-0.953 4.89859e-18 0.118125 rpy=0 -0 0 -> xyz=-0.953 -5.07838e-17 -0.118125 rpy=3.14159 -0 0.526654

Commit message: added traj optimization, the velocity at the end of traj opt drops suddenly

File: model_using_onshape_to_robot/cup_manipulator/cup_manipulator_obj.urdf (robot description, URDF)
Before this commit: robot cup_manipulator, 3 links, 2 joints
Links:
- link link1: mass 10.8153 -> 2.10
- link link2: mass 9.62243 -> 1.70
