Commit message: added isaac sim cup manipulator tendon model and webRTC client

File: model_using_onshape_to_robot/manipulator_cable_isaac/manipulator_cable.urdf (robot description, URDF)
Before this commit: robot manipulator_cable, 3 links, 2 joints
Links:
- link base_mate: geometry collision mesh filename=package://assets/base.stl; collision mesh filename=package://assets/pulle_htd_5m_12t.stl
- link link2_tendon: geometry collision mesh filename=package://assets/bearing_30x37.stl; collision mesh filename=package://assets/cup.stl
- link pulley_htd_5m_60t: geometry collision mesh filename=package://assets/623zz.stl; collision mesh filename=package://assets/623zz.stl

File: model_using_onshape_to_robot/manipulator_cable_isaac/manipulator_cable_obj.urdf (robot description, URDF)
Before this commit: robot manipulator_cable, 3 links, 2 joints
Links:
- link pulley_htd_5m_60t: geometry collision mesh filename=package://assets/base_kedua.obj; collision mesh filename=package://assets/gearbox_15_ratio.obj
